File: hardware/x35.kicad_pcb (KiCad board)
At the start: 2 copper layers, 15.2 x 27.9 mm, 15 parts, among them J1 USB_C_Receptacle_USB2.0_14P, J2 Conn_01x10, J3 Conn_01x10, SW1 SW_Push, U1 XC6206PxxxMR, U2 CH32X035x8x6

Commit message: Stash
Parts:
- removed JP2: Cut, PCM_ckl-misc:SolderJumper-2_Bridged_Pad_Small
- added G*** (x2): LOGO, LOGO, F.Cu at (118.8, 127.9)
- added G*** (x2): LOGO, LOGO, B.Cu at (118.8, 128.0)
- added REF**: Icy Electronics Logo, PCM_ckl-misc:Icy Electronics Logo, B.Cu at (116.2, 140.1)
- moved C2 41.6 mm to (116.5, 127.7)
- moved C3 41.6 mm to (116.8, 128.6)
- moved J2 41.6 mm to (125.8, 117.9)
- moved U1 41.6 mm to (116.0, 125.2)
- moved U2 41.6 mm to (119.5, 130.2)
- moved C1 41.6 mm to (115.5, 122.7)
- moved D2 41.6 mm to (115.6, 131.8)
- moved J1 41.6 mm to (118.8, 116.6)
- moved J3 41.6 mm to (111.8, 140.7)
- moved R1 41.6 mm to (120.6, 122.4)
- moved R2 41.6 mm to (118.5, 127.1)
- moved R3 41.6 mm to (117.3, 123.1)
- moved R5 41.6 mm to (116.6, 132.2)
- moved SW1 41.6 mm to (120.6, 124.5)
Connections:
- R5 pad 2: Net-(JP2-B) -> +3V3
Routing:
- net +3V3: track 15.6 -> 18.2 mm, vias 3 -> 4
- net Net-(JP2-B): track 1.65 -> 0.00 mm, vias 1 -> 0
Other:
- board text added: "5V 3V3 PA0 PA1 PA2 PA3 PA4 PA5"
- board text removed: "5V 3V3 PA0 PA1 PA2 PA3 PA4 PA5 GND"
