File: hardware/x35.kicad_sch (KiCad schematic)
At the start: 15 parts, among them J1 USB_C_Receptacle_USB2.0_14P, J2 Conn_01x10, J3 Conn_01x10, SW1 SW_Push, U1 XC6206PxxxMR, U2 CH32X035x8x6

Commit message: Stash
Parts:
- removed JP2: Cut, PCM_ckl-misc:SolderJumper-2_Bridged_Pad_Small, symbol Jumper:SolderJumper_2_Bridged
- U2: value CH32X035x8x6 -> CH32X035FxUx; footprint Package_DFN_QFN:QFN-20-1EP_3x3mm_P0.4mm_EP1.65x1.65mm_ThermalVias -> Package_DFN_QFN:QFN-20-1EP_3x3mm_P0.4mm_EP1.65x1.65mm; symbol here:CH32X035x8x6 -> here:CH32X035FxUx
Connections:
- net +3V3: now also R5.2
Changed lines of the file:
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@@
 	(wire
 		(pts
-			(xy 132.08 21.59) (xy 132.08 24.13)
+			(xy 132.08 22.86) (xy 132.08 24.13)
 		)
 		(stroke
@@
 	(wire
 		(pts
-			(xy 69.85 130.81) (xy 69.85 132.08)
-		)
-		(stroke
-			(width 0)
-			(type default)
-		)
-	)
-	(wire
-		(pts
 			(xy 48.26 157.48) (xy 55.88 157.48)
 		)
@@
 	(symbol
 		(lib_id "power:+3V3")
-		(at 132.08 21.59 0)
+		(at 132.08 22.86 0)
 		(unit 1)
 		(body_style 1)
@@
 		(dnp no)
 		(property "Reference" "#PWR014"
-			(at 132.08 25.4 0)
+			(at 132.08 26.67 0)
 			(hide yes)
 			(show_name no)
@@
 		)
 		(property "Value" "+3V3"
-			(at 132.08 16.51 0)
+			(at 132.08 17.78 0)
 			(show_name no)
 			(do_not_autoplace no)
@@
 		)
 		(property "Footprint" ""
-			(at 132.08 21.59 0)
+			(at 132.08 22.86 0)
 			(hide yes)
 			(show_name no)
@@
 		)
 		(property "Datasheet" ""
-			(at 132.08 21.59 0)
+			(at 132.08 22.86 0)
 			(hide yes)
 			(show_name no)
@@
 		)
 		(property "Description" "Power symbol creates a global label with name \"+3V3\""
-			(at 132.08 21.59 0)
+			(at 132.08 22.86 0)
 			(hide yes)
 			(show_name no)
@@
 	)
 	(symbol
-		(lib_id "here:CH32X035x8x6")
+		(lib_id "here:CH32X035FxUx")
 		(at 120.65 63.5 0)
 		(unit 1)
@@
 			)
 		)
-		(property "Value" "CH32X035x8x6"
+		(property "Value" "CH32X035FxUx"
 			(at 122.7933 44.45 0)
 			(show_name no)
@@
 			)
 		)
-		(property "Footprint" "Package_DFN_QFN:QFN-20-1EP_3x3mm_P0.4mm_EP1.65x1.65mm_ThermalVias"
+		(property "Footprint" "Package_DFN_QFN:QFN-20-1EP_3x3mm_P0.4mm_EP1.65x1.65mm"
 			(at 120.65 63.5 0)
 			(hide yes)
@@
 		)
 		(pin "17"
-			(alternate "D-")
 		)
 		(pin "20"
-			(alternate "CC2")
 		)
 		(pin "18"
-			(alternate "D+")
 		)
 		(pin "19"
-			(alternate "CC1")
 		)
 		(instances
@@
 	)
 	(symbol
-		(lib_id "Jumper:SolderJumper_2_Bridged")
-		(at 69.85 137.16 270)
-		(unit 1)
-		(body_style 1)
-		(exclude_from_sim no)
-		(in_bom no)
-		(on_board yes)
-		(in_pos_files yes)
-		(dnp yes)
-		(fields_autoplaced yes)
-		(property "Reference" "JP2"
-			(at 72.39 135.8899 90)
-			(show_name no)
-			(do_not_autoplace no)
-			(effects
-				(font
-					(size 1.27 1.27)
-				)
-				(justify left)
-			)
-		)
-		(property "Value" "Cut"
-			(at 72.39 138.4299 90)
-			(show_name no)
-			(do_not_autoplace no)
-			(effects
-				(font
-					(size 1.27 1.27)
-				)
-				(justify left)
-			)
-		)
-		(property "Footprint" "PCM_ckl-misc:SolderJumper-2_Bridged_Pad_Small"
-			(at 69.85 137.16 0)
-			(hide yes)
-			(show_name no)
-			(do_not_autoplace no)
-			(effects
-				(font
-					(size 1.27 1.27)
-				)
-			)
-		)
-		(property "Datasheet" ""
-			(at 63.5 137.16 0)
-			(hide yes)
-			(show_name no)
-			(do_not_autoplace no)
-			(effects
-				(font
-					(size 1.27 1.27)
-				)
-			)
-		)
-		(property "Description" "Solder Jumper, 2-pole, closed/bridged"
-			(at 64.77 137.16 0)
-			(hide yes)
-			(show_name no)
-			(do_not_autoplace no)
-			(effects
-				(font
-					(size 1.27 1.27)
-				)
-			)
-		)
-		(pin "2"
-		)
-		(pin "1"
-		)
-		(instances
-			(project "x35"
-				(path "/cb20e4d0-6e1a-4ffc-8ca5-f0a5d0ea8791"
-					(reference "JP2")
-					(unit 1)
-				)
-			)
-		)
-	)
-	(symbol
 		(lib_id "Connector:USB_C_Receptacle_USB2.0_14P")
 		(at 40.64 46.99 0)
@@
 	(symbol
 		(lib_id "power:+3V3")
-		(at 69.85 130.81 0)
+		(at 69.85 142.24 0)
 		(unit 1)
 		(body_style 1)
@@
 		(fields_autoplaced yes)
 		(property "Reference" "#PWR018"
-			(at 69.85 134.62 0)
+			(at 69.85 146.05 0)
 			(hide yes)
 			(show_name no)
@@
 		)
 		(property "Value" "+3V3"
-			(at 69.85 125.73 0)
+			(at 69.85 137.16 0)
 			(show_name no)
 			(do_not_autoplace no)
@@
 		)
 		(property "Footprint" ""
-			(at 69.85 130.81 0)
+			(at 69.85 142.24 0)
 			(hide yes)
 			(show_name no)
@@
 		)
 		(property "Datasheet" ""
-			(at 69.85 130.81 0)
+			(at 69.85 142.24 0)
 			(hide yes)
 			(show_name no)
@@
 		)
 		(property "Description" "Power symbol creates a global label with name \"+3V3\""
-			(at 69.85 130.81 0)
+			(at 69.85 142.24 0)
 			(hide yes)
 			(show_name no)
